File: pcb/video.kicad_sch (KiCad schematic)
At the start: 5 parts

Commit message: moved i2c mux to another page
Other:
- added sheet I2C Mux (schematics/i2c.kicad_sch)

Commit message: choose components and add footprints
Parts:
- gave numbers to parts that had none: 1
