File: pcb/video.kicad_sch (KiCad schematic)
At the start: 5 parts, among them J2 HDMI_A

Commit message: add shield
Parts:
- added U: (no value), symbol VGA:LOGO
- U: renamed from MK1; value Mounting_Hole_PAD -> (none); footprint Mounting_Holes:MountingHole_2.7mm -> (none)
- U: renamed from MK2; value Mounting_Hole_PAD -> (none); footprint Mounting_Holes:MountingHole_2.7mm -> (none)
- U: renamed from MK3; value Mounting_Hole_PAD -> (none); footprint Mounting_Holes:MountingHole_2.7mm -> (none)
- U: renamed from MK4; value Mounting_Hole_PAD -> (none); footprint Mounting_Holes:MountingHole_2.7mm -> (none)
- U: renamed from J2; value HDMI_A -> (none)
Changed lines of the file:
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@@
-(kicad_sch (version 20220126) (generator eeschema)
+(kicad_sch (version 20220404) (generator eeschema)
   (paper "A4")
   (title_block
@@
   (no_connect (at 24.13 241.3))
   (no_connect (at 24.13 226.06))
+  (polyline (pts (xy 53.34 113.03) (xy 68.58 113.03))
+    (stroke (width 0) (type default))
+  )
   (polyline (pts (xy 233.68 121.92) (xy 246.38 121.92))
     (stroke (width 0) (type default))
   )
+  (polyline (pts (xy 107.95 113.03) (xy 120.65 113.03))
+    (stroke (width 0) (type default))
+  )
+  (polyline (pts (xy 233.68 86.36) (xy 245.11 86.36))
+    (stroke (width 0) (type default))
+  )
   (polyline (pts (xy 53.34 83.82) (xy 68.58 83.82))
     (stroke (width 0) (type default))
   )
   (polyline (pts (xy 186.69 86.36) (xy 203.2 86.36))
-    (stroke (width 0) (type default))
-  )
-  (polyline (pts (xy 53.34 113.03) (xy 68.58 113.03))
-    (stroke (width 0) (type default))
-  )
-  (polyline (pts (xy 233.68 86.36) (xy 245.11 86.36))
-    (stroke (width 0) (type default))
-  )
-  (polyline (pts (xy 107.95 113.03) (xy 120.65 113.03))
     (stroke (width 0) (type default))
   )
@@
   (symbol (lib_id "EuroCard160mmX100mm_holes:Mounting_Hole_PAD-Mechanical") (at 24.13 223.52 0) (unit 1)
     (in_bom yes) (on_board yes)
-    (property "Reference" "MK1" (id 0) (at 26.67 222.2246 0)
-      (effects (font (size 1.27 1.27)) (justify left))
-    )
-    (property "Value" "Mounting_Hole_PAD" (id 1) (at 26.67 224.536 0)
-      (effects (font (size 1.27 1.27)) (justify left))
-    )
-    (property "Footprint" "Mounting_Holes:MountingHole_2.7mm" (id 2) (at 24.13 223.52 0)
+    (default_instance (reference "U") (unit 1) (value "") (footprint ""))
+    (property "Reference" "U" (id 0) (at 26.67 222.2246 0)
+      (effects (font (size 1.27 1.27)) (justify left))
+    )
+    (property "Value" "" (id 1) (at 26.67 224.536 0)
+      (effects (font (size 1.27 1.27)) (justify left))
+    )
+    (property "Footprint" "" (id 2) (at 24.13 223.52 0)
       (effects (font (size 1.27 1.27)) hide)
     )
@@
   (symbol (lib_id "EuroCard160mmX100mm_holes:Mounting_Hole_PAD-Mechanical") (at 24.13 231.14 0) (unit 1)
     (in_bom yes) (on_board yes)
-    (property "Reference" "MK2" (id 0) (at 26.67 229.8446 0)
-      (effects (font (size 1.27 1.27)) (justify left))
-    )
-    (property "Value" "Mounting_Hole_PAD" (id 1) (at 26.67 232.156 0)
-      (effects (font (size 1.27 1.27)) (justify left))
-    )
-    (property "Footprint" "Mounting_Holes:MountingHole_2.7mm" (id 2) (at 24.13 231.14 0)
+    (default_instance (reference "U") (unit 1) (value "") (footprint ""))
+    (property "Reference" "U" (id 0) (at 26.67 229.8446 0)
+      (effects (font (size 1.27 1.27)) (justify left))
+    )
+    (property "Value" "" (id 1) (at 26.67 232.156 0)
+      (effects (font (size 1.27 1.27)) (justify left))
+    )
+    (property "Footprint" "" (id 2) (at 24.13 231.14 0)
       (effects (font (size 1.27 1.27)) hide)
     )
@@
   (symbol (lib_id "EuroCard160mmX100mm_holes:Mounting_Hole_PAD-Mechanical") (at 24.13 238.76 0) (unit 1)
     (in_bom yes) (on_board yes)
-    (property "Reference" "MK3" (id 0) (at 26.67 237.4646 0)
-      (effects (font (size 1.27 1.27)) (justify left))
-    )
-    (property "Value" "Mounting_Hole_PAD" (id 1) (at 26.67 239.776 0)
-      (effects (font (size 1.27 1.27)) (justify left))
-    )
-    (property "Footprint" "Mounting_Holes:MountingHole_2.7mm" (id 2) (at 24.13 238.76 0)
+    (default_instance (reference "U") (unit 1) (value "") (footprint ""))
+    (property "Reference" "U" (id 0) (at 26.67 237.4646 0)
+      (effects (font (size 1.27 1.27)) (justify left))
+    )
+    (property "Value" "" (id 1) (at 26.67 239.776 0)
+      (effects (font (size 1.27 1.27)) (justify left))
+    )
+    (property "Footprint" "" (id 2) (at 24.13 238.76 0)
       (effects (font (size 1.27 1.27)) hide)
     )
@@
   (symbol (lib_id "EuroCard160mmX100mm_holes:Mounting_Hole_PAD-Mechanical") (at 24.13 246.38 0) (unit 1)
     (in_bom yes) (on_board yes)
-    (property "Reference" "MK4" (id 0) (at 26.67 245.0846 0)
-      (effects (font (size 1.27 1.27)) (justify left))
-    )
-    (property "Value" "Mounting_Hole_PAD" (id 1) (at 26.67 247.396 0)
-      (effects (font (size 1.27 1.27)) (justify left))
-    )
-    (property "Footprint" "Mounting_Holes:MountingHole_2.7mm" (id 2) (at 24.13 246.38 0)
+    (default_instance (reference "U") (unit 1) (value "") (footprint ""))
+    (property "Reference" "U" (id 0) (at 26.67 245.0846 0)
+      (effects (font (size 1.27 1.27)) (justify left))
+    )
+    (property "Value" "" (id 1) (at 26.67 247.396 0)
+      (effects (font (size 1.27 1.27)) (justify left))
+    )
+    (property "Footprint" "" (id 2) (at 24.13 246.38 0)
       (effects (font (size 1.27 1.27)) hide)
     )
@@
   (symbol (lib_id "VGA:LOGO") (at 250.19 86.36 90) (unit 1)
     (in_bom yes) (on_board yes) (fields_autoplaced)
-    (property "Reference" "#G1" (id 0) (at 245.3378 86.36 0)
-      (effects (font (size 1.27 1.27)) hide)
-    )
-    (property "Value" "LOGO" (id 1) (at 255.0422 86.36 0)
+    (default_instance (reference "U") (unit 1) (value "") (footprint ""))
+    (property "Reference" "U" (id 0) (at 245.3378 86.36 0)
+      (effects (font (size 1.27 1.27)) hide)
+    )
+    (property "Value" "" (id 1) (at 255.0422 86.36 0)
       (effects (font (size 1.27 1.27)) hide)
     )
@@
   (symbol (lib_id "Connector:HDMI_A") (at 246.38 121.92 0) (unit 1)
     (in_bom no) (on_board no) (fields_autoplaced)
-    (property "Reference" "J2" (id 0) (at 240.665 119.38 90)
+    (default_instance (reference "U") (unit 1) (value "") (footprint ""))
+    (property "Reference" "U" (id 0) (at 240.665 119.38 90)
       (effects (font (size 1.27 1.27)) (justify left) hide)
     )
-    (property "Value" "HDMI_A" (id 1) (at 256.54 119.888 0)
+    (property "Value" "" (id 1) (at 256.54 119.888 0)
       (effects (font (size 1.27 1.27)) (justify left) hide)
     )

Commit message: passed erc and drc
Parts:
- removed U (x2): (no value), symbol EuroCard160mmX100mm_holes:Mounting_Hole_PAD-Mechanical
Connections:
- no-connect marks 4 -> 2
