File: pcb/schematics/bus.kicad_sch (KiCad schematic)
At the start: 1 part, among them J1 09032967825

Commit message: add architecture diagramé
Connections:
- net +5V_Mod renamed +5V
Changed lines of the file:
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@@
+    (stroke (width 0) (type default))
+  )
+  (wire (pts (xy 163.83 19.05) (xy 163.83 31.75))
     (stroke (width 0) (type default))
   )
@@
     (stroke (width 0) (type default))
   )
-  (wire (pts (xy 82.55 16.51) (xy 82.55 46.99))
-    (stroke (width 0) (type default))
-  )
   (wire (pts (xy 86.36 62.23) (xy 69.85 62.23))
     (stroke (width 0) (type default))
@@
     (stroke (width 0) (type default))
   )
-  (wire (pts (xy 163.83 16.51) (xy 163.83 31.75))
-    (stroke (width 0) (type default))
-  )
   (wire (pts (xy 82.55 92.71) (xy 69.85 92.71))
     (stroke (width 0) (type default))
@@
     (stroke (width 0) (type default))
   )
+  (wire (pts (xy 82.55 19.05) (xy 82.55 46.99))
+    (stroke (width 0) (type default))
+  )
   (wire (pts (xy 86.36 31.75) (xy 86.36 62.23))
     (stroke (width 0) (type default))
@@
     (stroke (width 0) (type default))
   )
+  (wire (pts (xy 123.19 19.05) (xy 123.19 57.15))
+    (stroke (width 0) (type default))
+  )
   (wire (pts (xy 127 118.11) (xy 127 133.35))
     (stroke (width 0) (type default))
@@
     (stroke (width 0) (type default))
   )
-  (wire (pts (xy 123.19 16.51) (xy 123.19 57.15))
-    (stroke (width 0) (type default))
-  )
   (global_label "CONN_20" (shape input) (at 69.85 82.55 0)
     (effects (font (size 1.27 1.27)) (justify left))
@@
     )
   )
-  (global_label "+5V_Mod" (shape input) (at 163.83 16.51 0) (fields_autoplaced)
-    (effects (font (size 1.27 1.27)) (justify left))
-    (property "Intersheet References" "${INTERSHEET_REFS}" (id 0) (at 174.8307 16.4306 0)
-      (effects (font (size 1.27 1.27)) (justify left))
-    )
-  )
   (global_label "CONN_13" (shape input) (at 110.49 67.31 0)
     (effects (font (size 1.27 1.27)) (justify left))
@@
     )
   )
-  (global_label "+5V_Mod" (shape input) (at 82.55 16.51 0) (fields_autoplaced)
-    (effects (font (size 1.27 1.27)) (justify left))
-    (property "Intersheet References" "${INTERSHEET_REFS}" (id 0) (at 93.5507 16.4306 0)
-      (effects (font (size 1.27 1.27)) (justify left))
-    )
-  )
   (global_label "CONN_15" (shape input) (at 151.13 72.39 0)
     (effects (font (size 1.27 1.27)) (justify left))
     (property "Intersheet References" "${INTERSHEET_REFS}" (id 0) (at 163.4612 72.3106 0)
-      (effects (font (size 1.27 1.27)) (justify left))
-    )
-  )
-  (global_label "+5V_Mod" (shape input) (at 123.19 16.51 0) (fields_autoplaced)
-    (effects (font (size 1.27 1.27)) (justify left))
-    (property "Intersheet References" "${INTERSHEET_REFS}" (id 0) (at 134.1907 16.4306 0)
       (effects (font (size 1.27 1.27)) (justify left))
     )
@@
     (pin "95")
   )
+  (symbol (lib_id "power:+5V") (at 82.55 19.05 0) (unit 1)
+    (in_bom yes) (on_board yes) (fields_autoplaced)
+    (property "Reference" "#PWR?" (id 0) (at 82.55 22.86 0)
+      (effects (font (size 1.27 1.27)) hide)
+    )
+    (property "Value" "+5V" (id 1) (at 82.55 15.24 0)
+      (effects (font (size 1.27 1.27)))
+    )
+    (property "Footprint" "" (id 2) (at 82.55 19.05 0)
+      (effects (font (size 1.27 1.27)) hide)
+    )
+    (property "Datasheet" "" (id 3) (at 82.55 19.05 0)
+      (effects (font (size 1.27 1.27)) hide)
+    )
+    (pin "1")
+  )
   (symbol (lib_id "Conn-09031966821:09031966921") (at 153.67 26.67 0) (unit 1)
     (in_bom yes) (on_board yes)
@@
     (pin "96")
   )
+  (symbol (lib_id "power:+5V") (at 123.19 19.05 0) (unit 1)
+    (in_bom yes) (on_board yes) (fields_autoplaced)
+    (property "Reference" "#PWR?" (id 0) (at 123.19 22.86 0)
+      (effects (font (size 1.27 1.27)) hide)
+    )
+    (property "Value" "+5V" (id 1) (at 123.19 15.24 0)
+      (effects (font (size 1.27 1.27)))
+    )
+    (property "Footprint" "" (id 2) (at 123.19 19.05 0)
+      (effects (font (size 1.27 1.27)) hide)
+    )
+    (property "Datasheet" "" (id 3) (at 123.19 19.05 0)
+      (effects (font (size 1.27 1.27)) hide)
+    )
+    (pin "1")
+  )
+  (symbol (lib_id "power:+5V") (at 163.83 19.05 0) (unit 1)
+    (in_bom yes) (on_board yes) (fields_autoplaced)
+    (property "Reference" "#PWR?" (id 0) (at 163.83 22.86 0)
+      (effects (font (size 1.27 1.27)) hide)
+    )
+    (property "Value" "+5V" (id 1) (at 163.83 15.24 0)
+      (effects (font (size 1.27 1.27)))
+    )
+    (property "Footprint" "" (id 2) (at 163.83 19.05 0)
+      (effects (font (size 1.27 1.27)) hide)
+    )
+    (property "Datasheet" "" (id 3) (at 163.83 19.05 0)
+      (effects (font (size 1.27 1.27)) hide)
+    )
+    (pin "1")
+  )
   (symbol (lib_id "power:GND") (at 86.36 191.77 0) (mirror y) (unit 1)

Commit message: choose components and add footprints
Parts:
- J1: value 09032967825 -> 09031966921; Part Number 09032967825 -> 09031966921
Changed lines of the file:
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@@
       (effects (font (size 1.27 1.27)) (justify right))
     )
-    (property "Value" "09032967825" (id 1) (at 115.57 17.78 0)
+    (property "Value" "09031966921" (id 1) (at 115.57 17.78 0)
       (effects (font (size 1.27 1.27)) (justify right))
     )
@@
       (effects (font (size 1.27 1.27)) (justify left) hide)
     )
-    (property "Part Number" "09032967825" (id 26) (at 113.03 26.67 0)
+    (property "Part Number" "09031966921" (id 26) (at 113.03 26.67 0)
       (effects (font (size 1.27 1.27)) hide)
     )
@@
   (symbol (lib_id "power:+5V") (at 82.55 19.05 0) (unit 1)
     (in_bom yes) (on_board yes) (fields_autoplaced)
-    (property "Reference" "#PWR?" (id 0) (at 82.55 22.86 0)
+    (property "Reference" "#PWR092" (id 0) (at 82.55 22.86 0)
       (effects (font (size 1.27 1.27)) hide)
     )
@@
       (effects (font (size 1.27 1.27)) (justify right))
     )
-    (property "Value" "09032967825" (id 1) (at 156.21 17.78 0)
+    (property "Value" "09031966921" (id 1) (at 156.21 17.78 0)
       (effects (font (size 1.27 1.27)) (justify right))
     )
@@
       (effects (font (size 1.27 1.27)) (justify left) hide)
     )
-    (property "Part Number" "09032967825" (id 26) (at 153.67 26.67 0)
+    (property "Part Number" "09031966921" (id 26) (at 153.67 26.67 0)
       (effects (font (size 1.27 1.27)) hide)
     )
@@
   (symbol (lib_id "power:GND") (at 167.64 191.77 0) (mirror y) (unit 1)
     (in_bom yes) (on_board yes) (fields_autoplaced)
-    (property "Reference" "#PWR?" (id 0) (at 167.64 198.12 0)
+    (property "Reference" "#PWR097" (id 0) (at 167.64 198.12 0)
       (effects (font (size 1.27 1.27)) hide)
     )
@@
   (symbol (lib_id "power:GND") (at 127 191.77 0) (mirror y) (unit 1)
     (in_bom yes) (on_board yes) (fields_autoplaced)
-    (property "Reference" "#PWR?" (id 0) (at 127 198.12 0)
+    (property "Reference" "#PWR096" (id 0) (at 127 198.12 0)
       (effects (font (size 1.27 1.27)) hide)
     )
@@
       (effects (font (size 1.27 1.27)) (justify right))
     )
-    (property "Value" "09032967825" (id 1) (at 76.2 17.78 0)
+    (property "Value" "09031966921" (id 1) (at 76.2 17.78 0)
       (effects (font (size 1.27 1.27)) (justify right))
     )
@@
       (effects (font (size 1.27 1.27)) (justify left) hide)
     )
-    (property "Part Number" "09032967825" (id 26) (at 72.39 26.67 0)
+    (property "Part Number" "09031966921" (id 26) (at 72.39 26.67 0)
       (effects (font (size 1.27 1.27)) hide)
     )
@@
   (symbol (lib_id "power:+5V") (at 123.19 19.05 0) (unit 1)
     (in_bom yes) (on_board yes) (fields_autoplaced)
-    (property "Reference" "#PWR?" (id 0) (at 123.19 22.86 0)
+    (property "Reference" "#PWR093" (id 0) (at 123.19 22.86 0)
       (effects (font (size 1.27 1.27)) hide)
     )
@@
   (symbol (lib_id "power:+5V") (at 163.83 19.05 0) (unit 1)
     (in_bom yes) (on_board yes) (fields_autoplaced)
-    (property "Reference" "#PWR?" (id 0) (at 163.83 22.86 0)
+    (property "Reference" "#PWR094" (id 0) (at 163.83 22.86 0)
       (effects (font (size 1.27 1.27)) hide)
     )
@@
   (symbol (lib_id "power:GND") (at 86.36 191.77 0) (mirror y) (unit 1)
     (in_bom yes) (on_board yes) (fields_autoplaced)
-    (property "Reference" "#PWR?" (id 0) (at 86.36 198.12 0)
-      (effects (font (size 1.27 1.27)) hide)
-    )
+    (property "Reference" "#PWR095" (id 0) (at 86.36 198.12 0)
+      (effects (font (size 1.27 1.27)) hide)
+    )

Commit message: add a unified programming connector
Connections:
- net +5V: now also J1.13, J1.19, J1.40, J1.46, J1.67, J1.73, J1.94; no longer J1.15, J1.20, J1.42, J1.47, J1.69, J1.74, J1.96
- net CONN_1: now also J1.7; no longer J1.8
- net CONN_10: now also J1.19; no longer J1.21
- net CONN_11: now also J1.22; no longer J1.23
- net CONN_13: now also J1.25; no longer J1.26
- net CONN_14: now also J1.25; no longer J1.27
- net CONN_16: now also J1.28; no longer J1.30
- net CONN_17: now also J1.31; no longer J1.32
- net CONN_19: now also J1.34; no longer J1.35
- net CONN_2: now also J1.7; no longer J1.9
- net CONN_20: now also J1.34; no longer J1.36
- net CONN_22: now also J1.37; no longer J1.39
- net CONN_23: now also J1.40; no longer J1.41
- net CONN_25: now also J1.43; no longer J1.44
- net CONN_26: now also J1.43; no longer J1.45
- net CONN_28: now also J1.46; no longer J1.48
- net CONN_29: now also J1.49; no longer J1.50
- net CONN_31: now also J1.52; no longer J1.53
- net CONN_32: now also J1.52; no longer J1.54
- net CONN_34: now also J1.55; no longer J1.57
- net CONN_35: now also J1.58; no longer J1.59
- net CONN_37: now also J1.61; no longer J1.62
- net CONN_38: now also J1.61; no longer J1.63
- net CONN_4: now also J1.10; no longer J1.12
- net CONN_40: now also J1.64; no longer J1.66
- net CONN_41: now also J1.67; no longer J1.68
- net CONN_43: now also J1.70; no longer J1.71
- net CONN_44: now also J1.70; no longer J1.72
- net CONN_46: now also J1.73; no longer J1.75
- net CONN_47: now also J1.76; no longer J1.77
- net CONN_49: now also J1.79; no longer J1.80
- net CONN_5: now also J1.13; no longer J1.14
- net CONN_50: now also J1.79; no longer J1.81
- net CONN_52: now also J1.82; no longer J1.84
- net CONN_7: now also J1.16; no longer J1.17
- net CONN_8: now also J1.16; no longer J1.18
- net GND: now also J1.1, J1.10, J1.22, J1.28, J1.31, J1.37, J1.4, J1.4, J1.49, J1.55, J1.58, J1.64, J1.76, J1.82, J1.85, J1.85, J1.88, J1.91, J1.91, J1.94; no longer J1.11, J1.2, J1.24, J1.29, J1.33, J1.38, J1.5, J1.51, J1.56, J1.6, J1.60, J1.65, J1.78, J1.83, J1.86, J1.87, J1.90, J1.92, J1.93, J1.95
Changed lines of the file:
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@@
     )
   )
-  (symbol (lib_id "Conn-09031966821:09031966921") (at 113.03 26.67 0) (unit 2)
+  (symbol (lib_id "Conn-09031966821:09031966921") (at 113.03 26.67 0)
     (in_bom yes) (on_board yes)
     (property "Reference" "J1" (id 0) (at 115.57 15.24 0)
@@
     (pin "95")
   )
-  (symbol (lib_id "power:+5V") (at 82.55 19.05 0) (unit 1)
+  (symbol (lib_id "power:+5V") (at 82.55 19.05 0)
     (in_bom yes) (on_board yes) (fields_autoplaced)
     (property "Reference" "#PWR092" (id 0) (at 82.55 22.86 0)
@@
     (pin "1")
   )
-  (symbol (lib_id "Conn-09031966821:09031966921") (at 153.67 26.67 0) (unit 1)
+  (symbol (lib_id "Conn-09031966821:09031966921") (at 153.67 26.67 0)
     (in_bom yes) (on_board yes)
     (property "Reference" "J1" (id 0) (at 156.21 15.24 0)
@@
     (pin "94")
   )
-  (symbol (lib_id "power:GND") (at 167.64 191.77 0) (mirror y) (unit 1)
+  (symbol (lib_id "power:GND") (at 167.64 191.77 0) (mirror y)
     (in_bom yes) (on_board yes) (fields_autoplaced)
     (property "Reference" "#PWR097" (id 0) (at 167.64 198.12 0)
@@
     (pin "1")
   )
-  (symbol (lib_id "power:GND") (at 127 191.77 0) (mirror y) (unit 1)
+  (symbol (lib_id "power:GND") (at 127 191.77 0) (mirror y)
     (in_bom yes) (on_board yes) (fields_autoplaced)
     (property "Reference" "#PWR096" (id 0) (at 127 198.12 0)
@@
     (pin "1")
   )
-  (symbol (lib_id "Conn-09031966821:09031966921") (at 72.39 26.67 0) (unit 3)
+  (symbol (lib_id "Conn-09031966821:09031966921") (at 72.39 26.67 0)
     (in_bom yes) (on_board yes)
     (property "Reference" "J1" (id 0) (at 76.2 15.24 0)
@@
     (pin "96")
   )
-  (symbol (lib_id "power:+5V") (at 123.19 19.05 0) (unit 1)
+  (symbol (lib_id "power:+5V") (at 123.19 19.05 0)
     (in_bom yes) (on_board yes) (fields_autoplaced)
     (property "Reference" "#PWR093" (id 0) (at 123.19 22.86 0)
@@
     (pin "1")
   )
-  (symbol (lib_id "power:+5V") (at 163.83 19.05 0) (unit 1)
+  (symbol (lib_id "power:+5V") (at 163.83 19.05 0)
     (in_bom yes) (on_board yes) (fields_autoplaced)
     (property "Reference" "#PWR094" (id 0) (at 163.83 22.86 0)
@@
     (pin "1")
   )
-  (symbol (lib_id "power:GND") (at 86.36 191.77 0) (mirror y) (unit 1)
+  (symbol (lib_id "power:GND") (at 86.36 191.77 0) (mirror y)
     (in_bom yes) (on_board yes) (fields_autoplaced)
     (property "Reference" "#PWR095" (id 0) (at 86.36 198.12 0)

Commit message: add the programming controller
Connections:
- net +5V: now also J1.15, J1.20, J1.42, J1.47, J1.69, J1.74, J1.96; no longer J1.13, J1.19, J1.40, J1.46, J1.67, J1.73, J1.94
- net CONN_1: now also J1.8; no longer J1.7
- net CONN_10: now also J1.21; no longer J1.19
- net CONN_11: now also J1.23; no longer J1.22
- net CONN_13: now also J1.26; no longer J1.25
- net CONN_14: now also J1.27; no longer J1.25
- net CONN_16: now also J1.30; no longer J1.28
- net CONN_17: now also J1.32; no longer J1.31
- net CONN_19: now also J1.35; no longer J1.34
- net CONN_2: now also J1.9; no longer J1.7
- net CONN_20: now also J1.36; no longer J1.34
- net CONN_22: now also J1.39; no longer J1.37
- net CONN_23: now also J1.41; no longer J1.40
- net CONN_25: now also J1.44; no longer J1.43
- net CONN_26: now also J1.45; no longer J1.43
- net CONN_28: now also J1.48; no longer J1.46
- net CONN_29: now also J1.50; no longer J1.49
- net CONN_31: now also J1.53; no longer J1.52
- net CONN_32: now also J1.54; no longer J1.52
- net CONN_34: now also J1.57; no longer J1.55
- net CONN_35: now also J1.59; no longer J1.58
- net CONN_37: now also J1.62; no longer J1.61
- net CONN_38: now also J1.63; no longer J1.61
- net CONN_4: now also J1.12; no longer J1.10
- net CONN_40: now also J1.66; no longer J1.64
- net CONN_41: now also J1.68; no longer J1.67
- net CONN_43: now also J1.71; no longer J1.70
- net CONN_44: now also J1.72; no longer J1.70
- net CONN_46: now also J1.75; no longer J1.73
- net CONN_47: now also J1.77; no longer J1.76
- net CONN_49: now also J1.80; no longer J1.79
- net CONN_5: now also J1.14; no longer J1.13
- net CONN_50: now also J1.81; no longer J1.79
- net CONN_52: now also J1.84; no longer J1.82
- net CONN_7: now also J1.17; no longer J1.16
- net CONN_8: now also J1.18; no longer J1.16
- net GND: now also J1.11, J1.2, J1.24, J1.29, J1.33, J1.38, J1.5, J1.51, J1.56, J1.6, J1.60, J1.65, J1.78, J1.83, J1.86, J1.87, J1.92, J1.95; no longer J1.1, J1.10, J1.22, J1.28, J1.31, J1.37, J1.4, J1.4, J1.49, J1.55, J1.58, J1.64, J1.76, J1.82, J1.85, J1.85, J1.88, J1.91, J1.91, J1.94
- net TMS_CONN: now reaches J1.88
- new net RESET_CONN: J1.3
- new net TCK_CONN: J1.89
- new net TDI_CONN: J1.90
- new net TDO_CONN: J1.93
- no-connect marks 4 -> 1

Commit message: add shield
Parts:
- U: renamed from J1; value 09031966921 -> (none); footprint 09031966821:Harting-09031966921-0-0-0 -> (none)
Connections:
- net +5V: now also U.13, U.19, U.40, U.46, U.67, U.73, U.94; no longer U.15, U.20, U.42, U.47, U.69, U.74, U.96
- net CONN_1: now also U.7; no longer U.8
- net CONN_10: now also U.19; no longer U.21
- net CONN_11: now also U.22; no longer U.23
- net CONN_13: now also U.25; no longer U.26
- net CONN_14: now also U.25; no longer U.27
- net CONN_16: now also U.28; no longer U.30
- net CONN_17: now also U.31; no longer U.32
- net CONN_19: now also U.34; no longer U.35
- net CONN_2: now also U.7; no longer U.9
- net CONN_20: now also U.34; no longer U.36
- net CONN_22: now also U.37; no longer U.39
- net CONN_23: now also U.40; no longer U.41
- net CONN_25: now also U.43; no longer U.44
- net CONN_26: now also U.43; no longer U.45
- net CONN_28: now also U.46; no longer U.48
- net CONN_29: now also U.49; no longer U.50
- net CONN_31: now also U.52; no longer U.53
- net CONN_32: now also U.52; no longer U.54
- net CONN_34: now also U.55; no longer U.57
- net CONN_35: now also U.58; no longer U.59
- net CONN_37: now also U.61; no longer U.62
- net CONN_38: now also U.61; no longer U.63
- net CONN_4: now also U.10; no longer U.12
- net CONN_40: now also U.64; no longer U.66
- net CONN_41: now also U.67; no longer U.68
- net CONN_43: now also U.70; no longer U.71
- net CONN_44: now also U.70; no longer U.72
- net CONN_46: now also U.73; no longer U.75
- net CONN_47: now also U.76; no longer U.77
- net CONN_49: now also U.79; no longer U.80
- net CONN_5: now also U.13; no longer U.14
- net CONN_50: now also U.79; no longer U.81
- net CONN_52: now also U.82; no longer U.84
- net CONN_7: now also U.16; no longer U.17
- net CONN_8: now also U.16; no longer U.18
- net GND: now also U.1, U.10, U.22, U.28, U.31, U.37, U.4, U.4, U.49, U.55, U.58, U.64, U.76, U.82, U.85, U.85, U.91, U.94; no longer U.11, U.2, U.24, U.29, U.33, U.38, U.5, U.51, U.56, U.6, U.60, U.65, U.78, U.83, U.86, U.87, U.92, U.95
- net RESET_CONN: now also U.1; no longer U.3
- net TCK_CONN: now also U.88; no longer U.89
- net TDI_CONN: now also U.88; no longer U.90
- net TDO_CONN: now also U.91; no longer U.93
