File: pcb/schematics/dualport-ram.kicad_sch (KiCad schematic)
At the start: 4 parts, among them U11 S62LV256AL-45TLI

Commit message: add shield
Parts:
- U: renamed from U11; value S62LV256AL-45TLI -> (none); footprint Package_SO:TSOP-I-28_11.8x8mm_P0.55mm -> (none)
- U: renamed from R30; value 10k -> (none); footprint Resistor_SMD:R_0603_1608Metric -> (none)
- U: renamed from C95; value 100n -> (none); footprint Capacitor_SMD:C_0603_1608Metric -> (none)
- U: renamed from R29; value 10k -> (none); footprint Resistor_SMD:R_0603_1608Metric -> (none)
Changed lines of the file:
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@@
-(kicad_sch (version 20220126) (generator eeschema)
+(kicad_sch (version 20220404) (generator eeschema)
   (paper "A4")
   (junction (at 177.8 107.95) (diameter 0) (color 0 0 0 0)
@@
   (symbol (lib_id "power:GND") (at 151.13 120.65 0) (unit 1)
     (in_bom yes) (on_board yes) (fields_autoplaced)
-    (property "Reference" "#PWR0140" (id 0) (at 151.13 127 0)
-      (effects (font (size 1.27 1.27)) hide)
-    )
-    (property "Value" "GND" (id 1) (at 151.13 125.73 0)
+    (default_instance (reference "U") (unit 1) (value "") (footprint ""))
+    (property "Reference" "U" (id 0) (at 151.13 127 0)
+      (effects (font (size 1.27 1.27)) hide)
+    )
+    (property "Value" "" (id 1) (at 151.13 125.73 0)
       (effects (font (size 1.27 1.27)))
     )
@@
   (symbol (lib_id "IS62LV256:S62LV256AL-45TLI") (at 139.7 64.77 0) (unit 1)
     (in_bom yes) (on_board yes) (fields_autoplaced)
-    (property "Reference" "U11" (id 0) (at 141.5289 67.31 0)
-      (effects (font (size 1.27 1.27)) (justify left))
-    )
-    (property "Value" "S62LV256AL-45TLI" (id 1) (at 141.5289 69.85 0)
-      (effects (font (size 1.27 1.27)) (justify left))
-    )
-    (property "Footprint" "Package_SO:TSOP-I-28_11.8x8mm_P0.55mm" (id 2) (at 139.7 64.77 0)
+    (default_instance (reference "U") (unit 1) (value "") (footprint ""))
+    (property "Reference" "U" (id 0) (at 141.5289 67.31 0)
+      (effects (font (size 1.27 1.27)) (justify left))
+    )
+    (property "Value" "" (id 1) (at 141.5289 69.85 0)
+      (effects (font (size 1.27 1.27)) (justify left))
+    )
+    (property "Footprint" "" (id 2) (at 139.7 64.77 0)
       (effects (font (size 1.27 1.27)) hide)
     )
@@
   (symbol (lib_id "Device:R_Small") (at 177.8 100.33 0) (mirror y) (unit 1)
     (in_bom yes) (on_board yes) (fields_autoplaced)
-    (property "Reference" "R30" (id 0) (at 180.34 99.695 0)
-      (effects (font (size 1.27 1.27)) (justify right))
-    )
-    (property "Value" "10k" (id 1) (at 180.34 102.235 0)
-      (effects (font (size 1.27 1.27)) (justify right))
-    )
-    (property "Footprint" "Resistor_SMD:R_0603_1608Metric" (id 2) (at 177.8 100.33 0)
+    (default_instance (reference "U") (unit 1) (value "") (footprint ""))
+    (property "Reference" "U" (id 0) (at 180.34 99.695 0)
+      (effects (font (size 1.27 1.27)) (justify right))
+    )
+    (property "Value" "" (id 1) (at 180.34 102.235 0)
+      (effects (font (size 1.27 1.27)) (justify right))
+    )
+    (property "Footprint" "" (id 2) (at 177.8 100.33 0)
       (effects (font (size 1.27 1.27)) hide)
     )
@@
   (symbol (lib_id "Device:C_Small") (at 124.46 62.23 0) (mirror y) (unit 1)
     (in_bom yes) (on_board yes) (fields_autoplaced)
-    (property "Reference" "C95" (id 0) (at 121.92 61.6013 0)
-      (effects (font (size 1.27 1.27)) (justify left))
-    )
-    (property "Value" "100n" (id 1) (at 121.92 64.1413 0)
-      (effects (font (size 1.27 1.27)) (justify left))
-    )
-    (property "Footprint" "Capacitor_SMD:C_0603_1608Metric" (id 2) (at 124.46 62.23 0)
+    (default_instance (reference "U") (unit 1) (value "") (footprint ""))
+    (property "Reference" "U" (id 0) (at 121.92 61.6013 0)
+      (effects (font (size 1.27 1.27)) (justify left))
+    )
+    (property "Value" "" (id 1) (at 121.92 64.1413 0)
+      (effects (font (size 1.27 1.27)) (justify left))
+    )
+    (property "Footprint" "" (id 2) (at 124.46 62.23 0)
       (effects (font (size 1.27 1.27)) hide)
     )
@@
   (symbol (lib_id "power:+3V3") (at 177.8 96.52 0) (unit 1)
     (in_bom yes) (on_board yes) (fields_autoplaced)
-    (property "Reference" "#PWR0141" (id 0) (at 177.8 100.33 0)
-      (effects (font (size 1.27 1.27)) hide)
-    )
-    (property "Value" "+3V3" (id 1) (at 177.8 92.71 0)
+    (default_instance (reference "U") (unit 1) (value "") (footprint ""))
+    (property "Reference" "U" (id 0) (at 177.8 100.33 0)
+      (effects (font (size 1.27 1.27)) hide)
+    )
+    (property "Value" "" (id 1) (at 177.8 92.71 0)
       (effects (font (size 1.27 1.27)))
     )
@@
   (symbol (lib_id "Device:R_Small") (at 171.45 100.33 0) (mirror y) (unit 1)
     (in_bom yes) (on_board yes) (fields_autoplaced)
-    (property "Reference" "R29" (id 0) (at 168.91 99.695 0)
-      (effects (font (size 1.27 1.27)) (justify left))
-    )
-    (property "Value" "10k" (id 1) (at 168.91 102.235 0)
-      (effects (font (size 1.27 1.27)) (justify left))
-    )
-    (property "Footprint" "Resistor_SMD:R_0603_1608Metric" (id 2) (at 171.45 100.33 0)
+    (default_instance (reference "U") (unit 1) (value "") (footprint ""))
+    (property "Reference" "U" (id 0) (at 168.91 99.695 0)
+      (effects (font (size 1.27 1.27)) (justify left))
+    )
+    (property "Value" "" (id 1) (at 168.91 102.235 0)
+      (effects (font (size 1.27 1.27)) (justify left))
+    )
+    (property "Footprint" "" (id 2) (at 171.45 100.33 0)
       (effects (font (size 1.27 1.27)) hide)
     )
@@
   (symbol (lib_id "power:+3V3") (at 139.7 57.15 0) (unit 1)
     (in_bom yes) (on_board yes) (fields_autoplaced)
-    (property "Reference" "#PWR0137" (id 0) (at 139.7 60.96 0)
-      (effects (font (size 1.27 1.27)) hide)
-    )
-    (property "Value" "+3V3" (id 1) (at 139.7 53.34 0)
+    (default_instance (reference "U") (unit 1) (value "") (footprint ""))
+    (property "Reference" "U" (id 0) (at 139.7 60.96 0)
+      (effects (font (size 1.27 1.27)) hide)
+    )
+    (property "Value" "" (id 1) (at 139.7 53.34 0)
       (effects (font (size 1.27 1.27)))
     )
@@
   (symbol (lib_id "power:+3V3") (at 171.45 96.52 0) (unit 1)
     (in_bom yes) (on_board yes) (fields_autoplaced)
-    (property "Reference" "#PWR0142" (id 0) (at 171.45 100.33 0)
-      (effects (font (size 1.27 1.27)) hide)
-    )
-    (property "Value" "+3V3" (id 1) (at 171.45 92.71 0)
+    (default_instance (reference "U") (unit 1) (value "") (footprint ""))
+    (property "Reference" "U" (id 0) (at 171.45 100.33 0)
+      (effects (font (size 1.27 1.27)) hide)
+    )
+    (property "Value" "" (id 1) (at 171.45 92.71 0)
       (effects (font (size 1.27 1.27)))
     )
@@
   (symbol (lib_id "power:GND") (at 139.7 120.65 0) (unit 1)
     (in_bom yes) (on_board yes) (fields_autoplaced)
-    (property "Reference" "#PWR0139" (id 0) (at 139.7 127 0)
-      (effects (font (size 1.27 1.27)) hide)
-    )
-    (property "Value" "GND" (id 1) (at 139.7 125.73 0)
+    (default_instance (reference "U") (unit 1) (value "") (footprint ""))
+    (property "Reference" "U" (id 0) (at 139.7 127 0)
+      (effects (font (size 1.27 1.27)) hide)
+    )
+    (property "Value" "" (id 1) (at 139.7 125.73 0)
       (effects (font (size 1.27 1.27)))
     )
@@
   (symbol (lib_id "power:GND") (at 124.46 66.04 0) (mirror y) (unit 1)
     (in_bom yes) (on_board yes) (fields_autoplaced)
-    (property "Reference" "#PWR0138" (id 0) (at 124.46 72.39 0)
-      (effects (font (size 1.27 1.27)) hide)
-    )
-    (property "Value" "GND" (id 1) (at 124.46 71.12 0)
-      (effects (font (size 1.27 1.27)))
-    )
+    (default_instance (reference "U") (unit 1) (value "") (footprint ""))
+    (property "Reference" "U" (id 0) (at 124.46 72.39 0)
+      (effects (font (size 1.27 1.27)) hide)
+    )
+    (property "Value" "" (id 1) (at 124.46 71.12 0)
+      (effects (font (size 1.27 1.27)))
+    )
