File: pcb/schematics/i2c.kicad_sch (KiCad schematic)
At the start: 13 parts

Commit message: choose components and add footprints
Parts:
- C91, C92, C93: renamed from C?; footprint (none) -> Capacitor_SMD:C_0603_1608Metric; Part Number (none) -> EMK107B7104KA-T
- R21, R22, R23, R24, R25, R26, R27, R28: renamed from R?; footprint (none) -> Resistor_SMD:R_0603_1608Metric; Part Number (none) -> RC0603JR-0710KL
- U10: renamed from U?; footprint (none) -> Package_SO:TSSOP-8_3x3mm_P0.65mm; Part Number (none) -> NCA9306DPH
- U9: renamed from U?; footprint (none) -> Package_SO:TSSOP-8_3x3mm_P0.65mm; Part Number (none) -> PCA9540BDP,118

Commit message: add shield
Parts:
- U: renamed from U10; value NCA9306DPH -> (none); footprint Package_SO:TSSOP-8_3x3mm_P0.65mm -> (none)
- U: renamed from R26; value 10k -> (none); footprint Resistor_SMD:R_0603_1608Metric -> (none)
- U: renamed from C91; value 100n -> (none); footprint Capacitor_SMD:C_0603_1608Metric -> (none)
- U: renamed from R27; value 10k -> (none); footprint Resistor_SMD:R_0603_1608Metric -> (none)
- U: renamed from R28; value 10k -> (none); footprint Resistor_SMD:R_0603_1608Metric -> (none)
- U: renamed from R21; value 10k -> (none); footprint Resistor_SMD:R_0603_1608Metric -> (none)
- U: renamed from R22; value 10k -> (none); footprint Resistor_SMD:R_0603_1608Metric -> (none)
- U: renamed from R23; value 10k -> (none); footprint Resistor_SMD:R_0603_1608Metric -> (none)
- U: renamed from C93; value 100n -> (none); footprint Capacitor_SMD:C_0603_1608Metric -> (none)
- U: renamed from R24; value 10k -> (none); footprint Resistor_SMD:R_0603_1608Metric -> (none)
- U: renamed from R25; value 10k -> (none); footprint Resistor_SMD:R_0603_1608Metric -> (none)
- U: renamed from C92; value 100n -> (none); footprint Capacitor_SMD:C_0603_1608Metric -> (none)
- U: renamed from U9; value PCA9540BDP -> (none); footprint Package_SO:TSSOP-8_3x3mm_P0.65mm -> (none)
