File: pcb/schematics/power.kicad_sch (KiCad schematic)
At the start: 7 parts, among them U1 NCP115, U2 LP3853ESX-3.3/NOPB

Commit message: add shield
Parts:
- U: renamed from C4; value 10u -> (none); footprint Capacitor_SMD:C_0805_2012Metric -> (none)
- U: renamed from U1; value NCP115 -> (none); footprint NCP115ASN180T2G:NCP115ASN180T2G -> (none)
- U: renamed from C3; value 10u -> (none); footprint Capacitor_SMD:C_0805_2012Metric -> (none)
- U: renamed from U2; value LP3853ESX-3.3/NOPB -> (none); footprint LP3853ESX-3_3:LP3853ESX-3_3 -> (none)
- U: renamed from C1; value 10u -> (none); footprint Capacitor_SMD:C_0805_2012Metric -> (none)
- U: renamed from R1; value 10k -> (none); footprint Resistor_SMD:R_0603_1608Metric -> (none)
- U: renamed from C2; value 10u -> (none); footprint Capacitor_SMD:C_0805_2012Metric -> (none)

Commit message: passed erc and drc
Changed lines of the file:
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@@
   (junction (at 179.07 76.2) (diameter 0) (color 0 0 0 0)
   )
+  (junction (at 222.25 69.85) (diameter 0) (color 0 0 0 0)
+  )
   (junction (at 72.39 74.93) (diameter 0) (color 0 0 0 0)
   )
@@
     (stroke (width 0) (type default))
   )
-  (wire (pts (xy 137.16 74.93) (xy 137.16 68.58))
-    (stroke (width 0) (type default))
-  )
   (wire (pts (xy 63.5 68.58) (xy 63.5 74.93))
     (stroke (width 0) (type default))
   )
+  (wire (pts (xy 100.33 90.17) (xy 100.33 96.52))
+    (stroke (width 0) (type default))
+  )
   (wire (pts (xy 72.39 87.63) (xy 72.39 96.52))
     (stroke (width 0) (type default))
   )
-  (wire (pts (xy 222.25 68.58) (xy 222.25 76.2))
+  (wire (pts (xy 222.25 68.58) (xy 222.25 69.85))
     (stroke (width 0) (type default))
   )
@@
     (stroke (width 0) (type default))
   )
+  (wire (pts (xy 137.16 68.58) (xy 137.16 74.93))
+    (stroke (width 0) (type default))
+  )
   (wire (pts (xy 212.09 76.2) (xy 212.09 82.55))
     (stroke (width 0) (type default))
@@
     (stroke (width 0) (type default))
   )
+  (wire (pts (xy 222.25 69.85) (xy 222.25 76.2))
+    (stroke (width 0) (type default))
+  )
   (wire (pts (xy 72.39 74.93) (xy 72.39 82.55))
     (stroke (width 0) (type default))
@@
   )
   (wire (pts (xy 81.28 74.93) (xy 86.36 74.93))
-    (stroke (width 0) (type default))
-  )
-  (wire (pts (xy 100.33 90.17) (xy 100.33 96.52))
     (stroke (width 0) (type default))
   )
@@
       (effects (font (size 1.27 1.27)) hide)
     )
+    (pin "1")
+  )
+  (symbol (lib_id "power:PWR_FLAG") (at 222.25 69.85 90) (unit 1)
+    (in_bom yes) (on_board yes) (fields_autoplaced)
+    (default_instance (reference "#FLG") (unit 1) (value "PWR_FLAG") (footprint ""))
+    (property "Reference" "#FLG" (id 0) (at 220.345 69.85 0)
+      (effects (font (size 1.27 1.27)) hide)
+    )
+    (property "Value" "PWR_FLAG" (id 1) (at 218.44 70.485 90)
+      (effects (font (size 1.27 1.27)) (justify left))
+    )
+    (property "Footprint" "" (id 2) (at 222.25 69.85 0)
+      (effects (font (size 1.27 1.27)) hide)
+    )
+    (property "Datasheet" "~" (id 3) (at 222.25 69.85 0)
+      (effects (font (size 1.27 1.27)) hide)
+    )
